Commit message: updated_stereo

File: src/auv_slam/src/description/orca4_description.urdf (robot description, URDF)
Before this commit: robot orca4_ign, 11 links, 10 joints
Links:
- removed link camera_forward_link
- removed link left_camera_link
- removed link right_camera_link
- added link back_cam_link, mass 0.001; visual box size=0.02 0.02 0.02
- added link bottom_cam_link, mass 0.001; visual box size=0.02 0.02 0.02
- added link front_left_cam_link, mass 0.001; visual box size=0.02 0.02 0.02
- added link front_right_cam_link, mass 0.001; visual box size=0.02 0.02 0.02
- link imu_link: mass None -> 0.001
Joints:
- removed joint camera_forward_joint
- removed joint left_camera_joint
- removed joint right_camera_joint
- added joint back_cam_joint: type fixed, parent base_link, child back_cam_link, origin xyz=-0.24 0 0 rpy=0 0 3.141592
- added joint bottom_cam_joint: type fixed, parent base_link, child bottom_cam_link, origin xyz=0.1 0 -0.05 rpy=0 1.570796 0
- added joint front_left_cam_joint: type fixed, parent base_link, child front_left_cam_link, origin xyz=0.24 0.08 0 rpy=0 0 0
- added joint front_right_cam_joint: type fixed, parent base_link, child front_right_cam_link, origin xyz=0.24 -0.08 0 rpy=0 0 0
