Commit message: updated

File: src/auv_slam/src/description/varuna.urdf (robot description, URDF)
Before this commit: robot varuna_sauvc2026, 12 links, 11 joints
Links:
- link back_left_thrust: geometry collision mesh filename=package://varuna/meshes/back_left_thrust.STL; visual mesh filename=package://varuna/meshes/back_left_thrust.STL
- link back_right_thrust: geometry collision mesh filename=package://varuna/meshes/back_right_thrust.STL; visual mesh filename=package://varuna/meshes/back_right_thrust.STL
- link bottom_camera_link: geometry collision mesh filename=package://varuna/meshes/bottom_camera_link.STL; visual mesh filename=package://varuna/meshes/bottom_camera_link.STL
- link front_camera_link: geometry collision mesh filename=package://varuna/meshes/front_camera_link.STL; visual mesh filename=package://varuna/meshes/front_camera_link.STL
- link front_left_thrust: geometry collision mesh filename=package://varuna/meshes/front_left_thrust.STL; visual mesh filename=package://varuna/meshes/front_left_thrust.STL
- link front_right_thrust: geometry collision mesh filename=package://varuna/meshes/front_right_thrust.STL; visual mesh filename=package://varuna/meshes/front_right_thrust.STL
- link main_body: geometry collision mesh filename=package://varuna/meshes/main_body.STL; visual mesh filename=package://varuna/meshes/main_body.STL
- link surge_left_thrust: geometry collision mesh filename=package://varuna/meshes/surge_left_thrust.STL; visual mesh filename=package://varuna/meshes/surge_left_thrust.STL
- link surge_right_thrust: geometry collision mesh filename=package://varuna/meshes/surge_right_thrust.STL; visual mesh filename=package://varuna/meshes/surge_right_thrust.STL
- link sway_back_thrust: geometry collision mesh filename=package://varuna/meshes/sway_back_thrust.STL; visual mesh filename=package://varuna/meshes/sway_back_thrust.STL
- link sway_front_thrust: geometry collision mesh filename=package://varuna/meshes/sway_front_thrust.STL; visual mesh filename=package://varuna/meshes/sway_front_thrust.STL
